File: IR/KiCad/IR.kicad_pcb (KiCad board)
At the start: 2 copper layers, 17.8 x 15.2 mm, 4 parts, among them J1 Conn_01x06

Commit message: Deployed e8763eb with MkDocs version: 1.6.0
Parts:
- added REF**: MountingHole_3mm, MountingHole:MountingHole_3mm, F.Cu at (85.7, 50.8)
- moved IR1 10.4 mm to (96.1, 54.4)
- moved R1 10.2 mm to (80.3, 45.7), turned to 0 degrees
- moved D1 10.1 mm to (96.0, 48.0)
Routing:
- net GND: track 10.8 -> 22.9 mm, vias 0 -> 1
- net CLK: track 11.4 -> 21.9 mm
- net +3.3V: track 15.0 -> 23.8 mm
- net TX: track 12.0 -> 5.86 mm
Other:
- board size 17.8 x 15.2 mm -> 26.9 x 15.2 mm
- board text added: "IR"
- board text added: "IR Modul"
- board text added: "pmod.robotikabrno.cz/"

Commit message: Deployed 95a1413 with MkDocs version: 1.6.0
Parts:
- removed REF**: MountingHole_3mm, MountingHole:MountingHole_3mm
- added M3: MountingHole_3.2mm_M3, MountingHole:MountingHole_3.2mm_M3, F.Cu at (86.4, 50.8)
Routing:
- net GND: track 22.9 -> 1.37 mm, vias 1 -> 0
- added copper zone on B.Cu, net GND
- added copper zone on F.Cu, net GND
Changed lines of the file:
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@@
 		(at 96.0545 54.356 180)
 		(property "Reference" "IR1"
-			(at 2.4535 0.056 90)
+			(at 2.0745 0 90)
 			(layer "F.SilkS")
 			(effects
@@
 		(pad "1" thru_hole rect
 			(at 0 -2.54 180)
-			(size 2.5 1.8)
+			(size 2 1.6)
 			(drill 0.8)
 			(layers "*.Cu" "*.Mask")
@@
 		(pad "2" thru_hole oval
 			(at 0 0 180)
-			(size 2.5 1.8)
+			(size 2 1.6)
 			(drill 0.8)
 			(layers "*.Cu" "*.Mask")
@@
 		(pad "3" thru_hole oval
 			(at 0 2.54 180)
-			(size 2.5 1.8)
+			(size 2 1.6)
 			(drill 0.8)
 			(layers "*.Cu" "*.Mask")
@@
 		)
 	)
-	(footprint "MountingHole:MountingHole_3mm"
-		(layer "F.Cu")
-		(at 85.725 50.8)
-		(descr "Mounting Hole 3mm, no annular, generated by kicad-footprint-generator mountinghole.py")
-		(tags "mountinghole")
-		(property "Reference" "REF**"
-			(at 0 -3.95 0)
-			(layer "F.SilkS")
-			(hide yes)
-			(effects
-				(font
-					(size 1 1)
-					(thickness 0.15)
-				)
-			)
-		)
-		(property "Value" "MountingHole_3mm"
-			(at 0 3.95 0)
-			(layer "F.Fab")
-			(hide yes)
-			(effects
-				(font
-					(size 1 1)
-					(thickness 0.15)
-				)
-			)
-		)
-		(property "Datasheet" ""
-			(at 0 0 0)
-			(layer "F.Fab")
-			(hide yes)
-			(effects
-				(font
-					(size 1.27 1.27)
-					(thickness 0.15)
-				)
-			)
-		)
-		(property "Description" ""
-			(at 0 0 0)
-			(layer "F.Fab")
-			(hide yes)
-			(effects
-				(font
-					(size 1.27 1.27)
-					(thickness 0.15)
-				)
-			)
-		)
-		(attr exclude_from_pos_files exclude_from_bom)
-		(fp_circle
-			(center 0 0)
-			(end 3 0)
-			(stroke
-				(width 0.15)
-				(type solid)
-			)
-			(fill no)
-			(layer "Cmts.User")
-		)
-		(fp_circle
-			(center 0 0)
-			(end 3.25 0)
-			(stroke
-				(width 0.05)
-				(type solid)
-			)
-			(fill no)
-			(layer "F.CrtYd")
-		)
-		(fp_text user "${REFERENCE}"
-			(at 0 0 0)
-			(layer "F.Fab")
-			(effects
-				(font
-					(size 1 1)
-					(thickness 0.15)
-				)
-			)
-		)
-		(pad "" np_thru_hole circle
-			(at 0 0)
-			(size 3 3)
-			(drill 3)
-			(layers "*.Cu" "*.Mask")
-		)
-		(embedded_fonts no)
-	)
 	(footprint "Connector_PinHeader_2.54mm:PinHeader_1x06_P2.54mm_Horizontal"
 		(layer "F.Cu")
@@
 		)
 	)
+	(footprint "MountingHole:MountingHole_3.2mm_M3"
+		(layer "F.Cu")
+		(at 86.36 50.8)
+		(descr "Mounting Hole 3.2mm, M3, no annular, generated by kicad-footprint-generator mountinghole.py")
+		(tags "mountinghole M3")
+		(property "Reference" "M3"
+			(at 3.048 0 90)
+			(layer "F.SilkS")
+			(effects
+				(font
+					(size 1 1)
+					(thickness 0.15)
+				)
+			)
+		)
+		(property "Value" "MountingHole_3.2mm_M3"
+			(at 0 4.15 0)
+			(layer "F.Fab")
+			(hide yes)
+			(effects
+				(font
+					(size 1 1)
+					(thickness 0.15)
+				)
+			)
+		)
+		(property "Datasheet" ""
+			(at 0 0 0)
+			(layer "F.Fab")
+			(hide yes)
+			(effects
+				(font
+					(size 1.27 1.27)
+					(thickness 0.15)
+				)
+			)
+		)
+		(property "Description" ""
+			(at 0 0 0)
+			(layer "F.Fab")
+			(hide yes)
+			(effects
+				(font
+					(size 1.27 1.27)
+					(thickness 0.15)
+				)
+			)
+		)
+		(attr exclude_from_pos_files exclude_from_bom)
+		(fp_circle
+			(center 0 0)
+			(end 3.2 0)
+			(stroke
+				(width 0.15)
+				(type solid)
+			)
+			(fill no)
+			(layer "Cmts.User")
+		)
+		(fp_circle
+			(center 0 0)
+			(end 3.45 0)
+			(stroke
+				(width 0.05)
+				(type solid)
+			)
+			(fill no)
+			(layer "F.CrtYd")
+		)
+		(fp_text user "${REFERENCE}"
+			(at 0 0 0)
+			(layer "F.Fab")
+			(effects
+				(font
+					(size 1 1)
+					(thickness 0.15)
+				)
+			)
+		)
+		(pad "" np_thru_hole circle
+			(at 0 0)
+			(size 3.2 3.2)
+			(drill 3.2)
+			(layers "*.Cu" "*.Mask")
+		)
+		(embedded_fonts no)
+	)
 	(gr_poly
 		(pts
@@
 	)
 	(segment
-		(start 76.454 55.626)
-		(end 75.438 54.61)
-		(width 0.3)
-		(layer "F.Cu")
-		(net 2)
-	)
-	(segment
-		(start 91.694 55.626)
-		(end 76.454 55.626)
+		(start 74.93 52.07)
+		(end 75.692 52.07)
 		(width 0.3)
 		(layer "F.Cu")
-		(net 2)
-	)
-	(via
-		(at 91.694 55.626)
-		(size 0.6)
-		(drill 0.3)
-		(layers "F.Cu" "B.Cu")
-		(net 2)
-	)
-	(segment
-		(start 92.964 54.356)
-		(end 96.0545 54.356)
-		(width 0.3)
-		(layer "B.Cu")
-		(net 2)
-	)
-	(segment
-		(start 91.694 55.626)
-		(end 92.964 54.356)
-		(width 0.3)
-		(layer "B.Cu")
-		(net 2)
+		(net 3)
 	)
 	(segment
 		(start 77.851 54.229)
-		(end 92.71 54.229)
+		(end 90.297 54.229)
 		(width 0.3)
 		(layer "F.Cu")
@@
 	)
 	(segment
-		(start 74.93 52.07)
-		(end 75.692 52.07)
+		(start 92.964 56.896)
+		(end 96.0545 56.896)
 		(width 0.3)
 		(layer "F.Cu")
@@
 	)
 	(segment
-		(start 95.377 56.896)
-		(end 96.0545 56.896)
-		(width 0.3)
-		(layer "F.Cu")
-		(net 3)
-	)
-	(segment
-		(start 92.71 54.229)
-		(end 95.377 56.896)
+		(start 90.297 54.229)
+		(end 92.964 56.896)
 		(width 0.3)
 		(layer "F.Cu")
@@
 		(net 7)
 	)
+	(zone
+		(net 2)
+		(net_name "GND")
+		(layers "F.Cu" "B.Cu")
+		(hatch edge 0.5)
+		(connect_pads
+			(clearance 0.25)
+		)
+		(min_thickness 0.25)
+		(filled_areas_thickness no)
+		(fill yes
+			(thermal_gap 0.25)
+			(thermal_bridge_width 0.5)
+		)
+		(polygon
+			(pts
+				(xy 70.104 42.164) (xy 99.06 42.164) (xy 98.552 58.928) (xy 70.104 58.928)
+			)
+		)
+	)
 	(group ""
