File: MIC/KiCad/microphone.kicad_pcb (KiCad board)
At the start: 2 copper layers, 43.5 x 34 mm, 17 parts, among them J1 Conn_01x06_Pin, U1 LMV321

Commit message: Deployed 95a1413 with MkDocs version: 1.6.0
Parts:
- moved J1 0.58 mm to (141.5, 95.1)
Routing:
- net +3V3: track 46.7 -> 47.5 mm
- net Net-(J1-Pin_6): track 35.2 -> 35.8 mm
Other:
- board text added: "pmod.robotikabrno.cz/"
- board text removed: "https://pmod.robotikabrno.cz/pmod/"
Changed lines of the file:
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@@
 			(psa4output no)
 			(plot_black_and_white yes)
-			(plotinvisibletext no)
 			(sketchpadsonfab no)
 			(plotpadnumbers no)
@@
 		)
 		(property "Value" "1uF"
-			(at 2.5 2.2 90)
+			(at -2.448 -0.025 90)
 			(layer "F.Fab")
 			(effects
@@
 	(footprint "Connector_PinHeader_2.54mm:PinHeader_1x06_P2.54mm_Horizontal"
 		(layer "F.Cu")
-		(at 141 95.3)
+		(at 141.548 95.123)
 		(descr "Through hole angled pin header, 1x06, 2.54mm pitch, 6mm pin length, single row")
 		(tags "Through hole angled pin header THT 1x06 2.54mm single row")
@@
 		)
 		(property "Value" "10k"
-			(at 5.08 2.37 90)
+			(at 7.488 0 90)
 			(layer "F.Fab")
 			(effects
@@
 		(layer "Edge.Cuts")
 	)
-	(gr_text "https://pmod.robotikabrno.cz/pmod/"
-		(at 104.14 116.84 90)
+	(gr_text "pmod.robotikabrno.cz/"
+		(at 104.648 111.252 90)
 		(layer "F.SilkS")
 		(effects
@@
 	)
 	(gr_text "MIC"
-		(at 104.1654 88.392 90)
+		(at 104.902 94.234 90)
 		(layer "F.SilkS")
 		(effects
@@
 	)
 	(segment
-		(start 139 97)
-		(end 140.7 95.3)
+		(start 132.08 88.5)
+		(end 133.712 88.5)
 		(width 0.5)
 		(layer "F.Cu")
@@
 	)
 	(segment
-		(start 134.12 88.5)
-		(end 141 95.38)
+		(start 133.712 88.5)
+		(end 140.335 95.123)
 		(width 0.5)
 		(layer "F.Cu")
@@
 	)
 	(segment
-		(start 140.7 95.3)
-		(end 141 95.3)
+		(start 129.5 88.5)
+		(end 132.08 88.5)
 		(width 0.5)
 		(layer "F.Cu")
@@
 	)
 	(segment
-		(start 129.5 88.5)
-		(end 132.08 88.5)
+		(start 132.58 114.5)
+		(end 135.5 114.5)
 		(width 0.5)
 		(layer "F.Cu")
@@
 	)
 	(segment
-		(start 135.5 114.5)
-		(end 139 111)
+		(start 141.548 95.123)
+		(end 141.371 95.3)
 		(width 0.5)
 		(layer "F.Cu")
@@
 	)
 	(segment
-		(start 139 111)
-		(end 139 97)
+		(start 126.05 91.95)
+		(end 126.05 94.8625)
 		(width 0.5)
 		(layer "F.Cu")
@@
 	)
 	(segment
-		(start 132.08 88.5)
-		(end 134.12 88.5)
+		(start 139 96.458)
+		(end 140.335 95.123)
 		(width 0.5)
 		(layer "F.Cu")
@@
 	)
 	(segment
-		(start 126.05 91.95)
-		(end 126.05 94.8625)
+		(start 141.371 95.3)
+		(end 141 95.3)
+		(width 0.5)
+		(layer "F.Cu")
+		(net 5)
+	)
+	(segment
+		(start 135.5 114.5)
+		(end 139 111)
+		(width 0.5)
+		(layer "F.Cu")
+		(net 5)
+	)
+	(segment
+		(start 139 111)
+		(end 139 96.458)
 		(width 0.5)
 		(layer "F.Cu")
@@
 	)
 	(segment
-		(start 132.58 114.5)
-		(end 135.5 114.5)
+		(start 140.335 95.123)
+		(end 141.548 95.123)
 		(width 0.5)
 		(layer "F.Cu")
@@
 	)
 	(segment
+		(start 141.177 107.823)
+		(end 141.548 107.823)
+		(width 0.5)
+		(layer "B.Cu")
+		(net 7)
+	)
+	(segment
 		(start 131 101.5)
 		(end 131 95)
@@
 	)
 	(segment
-		(start 137 112)
-		(end 141 108)
+		(start 129 109.5)
+		(end 131.5 112)
 		(width 0.5)
 		(layer "B.Cu")
@@
 	)
 	(segment
-		(start 126.5 106)
-		(end 131 101.5)
+		(start 137 112)
+		(end 141.177 107.823)
 		(width 0.5)
 		(layer "B.Cu")
@@
 	)
 	(segment
-		(start 129 109.5)
-		(end 131.5 112)
+		(start 126.5 106)
+		(end 131 101.5)
 		(width 0.5)
 		(layer "B.Cu")
@@
 	)
 	(segment
-		(start 140.625 100.65)
-		(end 140.35 100.65)
-		(width 0.2)
-		(layer "F.Cu")
-		(net 9)
-	)
-	(segment
