File: r-encoder/KiCad/RotaryEncoder.kicad_pcb (KiCad board)
At the start: 2 copper layers, 39 x 39 mm, 15 parts, among them J1 Conn_01x06, U1 PEC11R-4325F-S0012

Commit message: Deployed 95a1413 with MkDocs version: 1.6.0
Parts:
- J1: footprint Connector_PinHeader_2.54mm:PinHeader_1x06_P2.54mm_Vertical -> Connector_PinHeader_2.54mm:PinHeader_1x06_P2.54mm_Horizontal
- moved J1 12.8 mm to (110.2, 80.1), turned to 180 degrees
Connections:
- J1 pad 1: A -> unconnected-(J1-Pin_1-Pad1)
- J1 pad 2: B -> BTN
- J1 pad 3: BTN -> B
- J1 pad 4: unconnected-(J1-Pin_4-Pad4) -> A
Routing:
- net GND: track 9.76 -> 0.00 mm, vias 17 -> 15
- net A: track 12.2 -> 17.3 mm
- net B: track 21.1 -> 17.7 mm
- net VCC: track 55.4 -> 54.8 mm
- net BTN: track 32.9 -> 33.2 mm, vias 0 -> 1
