File: r-encoder/KiCad/RotaryEncoder.kicad_sch (KiCad schematic)
At the start: 9 parts, among them J1 Conn_01x06, SW1 RotaryEncoder_Switch

Commit message: Deployed 95a1413 with MkDocs version: 1.6.0
Parts:
- removed SW1: RotaryEncoder_Switch, symbol Device:RotaryEncoder_Switch
- added C3: 0.01uF, Capacitor_THT:C_Disc_D3.8mm_W2.6mm_P2.50mm, symbol Device:C
- added H1, H2, H3, H4: MountingHole, MountingHole:MountingHole_3.2mm_M3, symbol Mechanical:MountingHole
- added R6: 10K, Resistor_THT:R_Axial_DIN0204_L3.6mm_D1.6mm_P5.08mm_Horizontal, symbol Device:R
- added U1: PEC11R-4325F-S0012, SamacSys_Parts:PEC11R4325FS0012, symbol SamacSys_Parts:PEC11R-4325F-S0012
- C1, C2: footprint (none) -> Capacitor_THT:C_Disc_D3.8mm_W2.6mm_P2.50mm
- J1: footprint (none) -> Connector_PinHeader_2.54mm:PinHeader_1x06_P2.54mm_Horizontal
- R1, R2, R3, R4, R5: footprint (none) -> Resistor_THT:R_Axial_DIN0204_L3.6mm_D1.6mm_P5.08mm_Horizontal
Connections:
- net A: now also C1.2, J1.4 (Pin_4), R3.2; no longer J1.3 (Pin_3), R1.2, R3.1
- net B: now also C2.2, J1.3 (Pin_3), R4.1; no longer J1.4 (Pin_4), R2.2, R4.2
- net BTN: now also J1.2 (Pin_2), C3.1, R6.2; no longer J1.5 (Pin_5), R5.1
- net GND: now also J1.5 (Pin_5), C3.2, U1.2 (NO), U1.3 (MH1), U1.4 (MH2), U1.C1 (C_COMMON); no longer J1.2 (Pin_2)
- net VCC: now also J1.6 (Pin_6); no longer J1.1 (Pin_1)
- new net: R5.1, R6.1, U1.1 (COM)
- new net: R2.2, R4.2, U1.B1 (B_CHANNEL)
- new net: R1.2, R3.1, U1.A1 (A_CHANNEL)
Other:
- moved on the sheet: J1, R5
